File: AS5047P.kicad_sch (KiCad schematic)
At the start: 25 parts, among them J1 Conn_01x06, J2 Conn_01x05, J3 Conn_01x05, U1 AS5047D

Commit message: 增加LED电路
Parts:
- added D1: LED_Small, symbol Device:LED_Small
- added R21: 1K, symbol Device:R_Small_US
Connections:
- net +3.3V: now also R21.2
- net GND: now also D1.1 (K)
- new net: D1.2 (A), R21.1
